File: OpenX3/untitled.brd (EAGLE design)
At the start: 100 x 80 mm, 20 parts, among them J1 SM20B-SRDS-G-TF(LF)(SN), U1 LC4256V-75TN100CTQFP100-L, U2 AM29F016D-70EF

Commit message: more work
Parts:
- added J2: SM12B-SRSS-TB(LF)(SN), SM12B-SRSS-TB:CONN_SM12B-SRSS-TB(LF)(SN)
- added R1, R2, R3, R4: UM6K31NFHATCNTRANS_UM6J1-L, UM6K31NFHA:TRANS_UM6J1-L
- added R5, R6: 10k, SparkFun-Resistors:0603
- added R7: 0, SparkFun-Resistors:0603
- added RN1, RN2: 10k, resistor-dil:0603-ARV
- added RN3: 100, resistor-dil:0603-ARV
- added U3: SST39SF020A-55-4C-WHE, SST39SF020A-55-4C-WHE:TSOP32_WH_SST
- moved PAD9 91.4 mm to (20.3, 2.54)
- moved PAD8 90.4 mm to (22.9, 2.54)
- moved PAD7 89.5 mm to (25.4, 2.54)
- moved PAD6 88.5 mm to (27.9, 2.54)
- moved PAD5 87.5 mm to (30.5, 2.54)
- moved PAD4 86.5 mm to (33.0, 2.54)
- moved PAD3 85.5 mm to (35.6, 2.54)
- moved PAD2 84.6 mm to (38.1, 2.54)
- moved PAD1 83.6 mm to (40.6, 2.54)
- moved JP1 80.7 mm to (47.0, 11.4), turned to 90 degrees
- moved PAD15 74.0 mm to (5.08, 2.54)
- moved PAD14 73.0 mm to (7.62, 2.54)
- moved PAD10 72.0 mm to (17.8, 2.54)
- moved PAD13 72.0 mm to (10.2, 2.54)
- moved U1 71.2 mm to (31.8, 22.9), turned to 90 degrees
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Connections:
- net N$1 renamed A19
- net N$26 renamed OE#
- net N$3 renamed LAD2
- net N$34 renamed A20
- net N$4 renamed LAD1
- net N$5 renamed LAD0
- net N$6 renamed LAD3
- net N$7 renamed A18
- removed net GND_4: U1.18
- removed net N$10: U1.92, U2.7
- removed net N$11: U1.93, U2.8
- removed net N$12: U1.94, U2.9
- removed net N$13: U1.97, U2.10
- removed net N$14: U1.17, U2.11
- removed net N$15: U1.98, U2.15
- removed net N$16: U1.99, U2.16
- removed net N$18: U1.3, U2.18
- removed net N$19: U1.4, U2.19
- removed net N$20: U1.5, U2.20
- removed net N$21: U1.6, U2.21
- removed net N$22: U1.8, U2.22
- removed net N$23: U1.9, U2.27
- removed net N$24: U1.10, U2.28
- removed net N$25: U1.11, U2.29
- removed net N$27: U1.12, U2.31
- removed net N$28: U1.72, U2.32
- removed net N$30: U1.60, U2.38
- removed net N$31: U1.61, U2.34
- removed net N$32: U1.59, U2.39
- removed net N$33: U1.50, U2.40
- removed net N$35: U1.13, U2.30
- removed net N$36: U1.15, U2.44
- removed net N$38: U1.49, U2.41
- removed net N$8: U1.87, U2.5
- removed net N$9: U1.91, U2.6
- new net 3V3: JP1.9, R5.2, R6.1
- new net A0: U1.13, U2.30, U3.20
- new net A1: U1.11, U2.29, U3.19
- new net A10: U1.99, U2.16, U3.31
- new net A11: U1.98, U2.15, U3.1
- new net A12: U1.97, U2.10, U3.12
- new net A13: U1.94, U2.9, U3.4
- new net A14: U1.93, U2.8, U3.5
- new net A15: U1.92, U2.7, U3.11
- new net A16: U1.91, U2.6, U3.10
- new net A17: U1.87, U2.5, U3.6
- new net A2: U1.10, U2.28, U3.18
- new net A3: U1.9, U2.27, U3.17
- new net A4: U1.8, U2.22, U3.16
- new net A5: U1.6, U2.21, U3.15
- new net A6: U1.5, U2.20, U3.14
- new net A7: U1.4, U2.19, U3.13
- new net A8: U1.3, U2.18, U3.3
- new net BUFLCE#: U1.19, U3.30
- new net D0: JP1.4, R2.1
- new net DQ0: U1.12, U2.31, U3.21
- new net DQ1: U1.72, U2.32, U3.22
- new net DQ3: U1.61, U2.34, U3.25
- new net DQ4: U1.60, U2.38, U3.26
- new net DQ5: U1.59, U2.39, U3.27
- new net DQ6: U1.50, U2.40, U3.28
- new net DQ7: U1.49, U2.41, U3.29
- new net MNFLCE#: U1.17, U2.11, U3.32
- new net N$56: R1.3, R1.6
- new net N$57: R1.2
- new net N$58: R1.5
- new net N$59: R1.4, R5.1, U1.39
- new net N$61: R1.1, R6.2, U1.41
- new net N$62: R2.2, U1.22
- new net N$63: R2.5, U1.20
- new net N$65: R2.3, R2.6, U1.18
- new net N$66: J2.10, RN3.5
- new net N$67: R3.1, R3.4, R4.1, R4.4, R7.2, RN2.1, RN2.2, RN2.3, RN2.4, U1.23, U1.27, U1.28, U1.29
- new net N$68: R3.2, RN1.5
- new net N$69: R3.5, RN1.6
- new net N$70: R4.5, RN1.7
- new net N$71: R4.2, RN1.8
- new net N$72: R3.6, RN3.4
- new net N$73: R3.3, RN3.3
- new net N$74: R4.3, RN3.2
- new net N$75: R4.6, RN3.1
- new net N$76: RN1.4
- new net N$77: RN1.3
- new net N$78: RN1.1, U1.31
- new net N$79: RN1.2, U1.30
- new net N$80: J2.9, RN3.6
- new net N$81: J2.8, RN3.7
- new net N$82: J2.7, RN3.8
- new net N$83: J2.6, RN2.5
- new net N$84: J2.5, RN2.6
- new net N$85: J2.4, RN2.7
- new net N$86: J2.3, RN2.8
- new net N$87: J2.1, R7.1
- new net VDD: U3.8
- new net WE#: U1.15, U2.44, U3.7
- net N$17: now also U3.2
- net N$29: now also U3.23
- net N$54: now also R2.4
- net VSS: now also U3.24
Routing:
- net DQ3: track 0.00 -> 142.1 mm, vias 0 -> 4
- net WE#: track 0.00 -> 136.9 mm, vias 0 -> 10
- net DQ4: track 0.00 -> 126.6 mm, vias 0 -> 5
- net DQ5: track 0.00 -> 108.0 mm, vias 0 -> 8
- net DQ6: track 0.00 -> 108.0 mm, vias 0 -> 5
- net DQ7: track 0.00 -> 95.9 mm, vias 0 -> 6
- net A2: track 0.00 -> 95.1 mm, vias 0 -> 10
- net N$42: track 0.00 -> 80.0 mm, vias 0 -> 9
- net VSS: track 0.00 -> 76.5 mm, vias 0 -> 4
- net MNFLCE#: track 0.00 -> 76.3 mm, vias 0 -> 6
- net A3: track 0.00 -> 73.0 mm, vias 0 -> 4
- net A1: track 0.00 -> 69.1 mm, vias 0 -> 7
- net N$41: track 0.00 -> 66.5 mm, vias 0 -> 9
- net A0: track 0.00 -> 60.0 mm, vias 0 -> 5
- net A11: track 0.00 -> 56.5 mm, vias 0 -> 5
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Other:
- board size 100 x 80 mm -> 50.5 x 45.7 mm
