File: OpenX3/untitled.brd (EAGLE design)
At the start: 46.7 x 49.1 mm, 50 parts, among them IC1 24AA256SN, J1 SM20B-SRDS-G-TF(LF)(SN), J2 SM12B-SRSS-TB(LF)(SN), J3 53398-0271, J4 1734260-3, U1 LC4256V-75TN100CTQFP100-L, U2 AM29F016D-70EF, U3 AM29F002BB90EI

Commit message: review ERC warnings; fix two missing junctions; one missing connection to GND on CPLD pin 18
Connections:
- removed net N$65: R2.3, R2.6, U1.18
- net GND: now also R2.3, R2.6, U1.18
Changed lines of the file:
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@@
 <wire x1="43.18" y1="4.318" x2="32.7152" y2="6.97" width="0" layer="19" extent="1-1"/>
-</signal>
-<signal name="N$65">
-<contactref element="R2" pad="3"/>
-<contactref element="R2" pad="6"/>
-<contactref element="U1" pad="18"/>
-<wire x1="32.7152" y1="8.27" x2="29.17" y2="16.55445" width="0" layer="19" extent="1-1"/>
-<wire x1="30.7848" y1="6.97" x2="32.7152" y2="8.27" width="0" layer="19" extent="1-1"/>
 </signal>
 <signal name="N$70">
@@
 <vertex x="-1.27" y="-1.27"/>
 </polygon>
+<contactref element="R2" pad="3"/>
+<contactref element="R2" pad="6"/>
+<contactref element="U1" pad="18"/>
+<wire x1="37.63" y1="41.152" x2="37.63" y2="40.652" width="0" layer="19" extent="1-1"/>
+<wire x1="40.73" y1="35.52" x2="37.63" y2="40.652" width="0" layer="19" extent="1-1"/>
+<wire x1="38.1" y1="32.5" x2="40.73" y2="35.52" width="0" layer="19" extent="1-1"/>
+<wire x1="37.6428" y1="27.94" x2="38.1" y2="32.5" width="0" layer="19" extent="1-16"/>
+<wire x1="37.6428" y1="25.4" x2="37.6428" y2="27.94" width="0" layer="19" extent="16-16"/>
+<wire x1="37.6428" y1="22.86" x2="37.6428" y2="25.4" width="0" layer="19" extent="16-16"/>
+<wire x1="37.6428" y1="20.32" x2="37.6428" y2="22.86" width="0" layer="19" extent="16-16"/>
+<wire x1="34.24555" y1="28.13" x2="37.6428" y2="27.94" width="0" layer="19" extent="1-16"/>
+<wire x1="34.24555" y1="21.13" x2="37.6428" y2="20.32" width="0" layer="19" extent="1-16"/>
+<wire x1="34.24555" y1="18.13" x2="34.24555" y2="21.13" width="0" layer="19" extent="1-1"/>
+<wire x1="36.83" y1="15.99" x2="34.24555" y2="18.13" width="0" layer="19" extent="1-1"/>
+<wire x1="32.67" y1="31.70555" x2="34.24555" y2="28.13" width="0" layer="19" extent="1-1"/>
+<wire x1="29.67" y1="31.70555" x2="32.67" y2="31.70555" width="0" layer="19" extent="1-1"/>
+<wire x1="29.17" y1="16.55445" x2="34.24555" y2="18.13" width="0" layer="19" extent="1-1"/>
+<wire x1="24.17" y1="31.70555" x2="29.67" y2="31.70555" width="0" layer="19" extent="1-1"/>
+<wire x1="19.09445" y1="30.13" x2="24.17" y2="31.70555" width="0" layer="19" extent="1-1"/>
+<wire x1="19.09445" y1="27.13" x2="19.09445" y2="30.13" width="0" layer="19" extent="1-1"/>
+<wire x1="23.67" y1="16.55445" x2="29.17" y2="16.55445" width="0" layer="19" extent="1-1"/>
+<wire x1="20.67" y1="16.55445" x2="23.67" y2="16.55445" width="0" layer="19" extent="1-1"/>
+<wire x1="19.09445" y1="20.13" x2="20.67" y2="16.55445" width="0" layer="19" extent="1-1"/>
+<wire x1="43.24" y1="26.289" x2="37.6428" y2="25.4" width="0" layer="19" extent="1-16"/>
+<wire x1="43.18" y1="14.478" x2="36.83" y2="15.99" width="0" layer="19" extent="1-1"/>
+<wire x1="32.7152" y1="8.27" x2="36.83" y2="15.99" width="0" layer="19" extent="1-1"/>
+<wire x1="30.7848" y1="6.97" x2="32.7152" y2="8.27" width="0" layer="19" extent="1-1"/>
+<wire x1="11.01" y1="15.24" x2="19.09445" y2="20.13" width="0" layer="19" extent="1-1"/>
+<wire x1="2.54" y1="17.56" x2="11.01" y2="15.24" width="0" layer="19" extent="1-1"/>
+<wire x1="2.096" y1="12.58" x2="2.54" y2="17.56" width="0" layer="19" extent="1-1"/>
+<wire x1="3.9287" y1="23.44" x2="2.54" y2="17.56" width="0" layer="19" extent="1-1"/>
+<wire x1="43.18" y1="1.778" x2="32.7152" y2="8.27" width="0" layer="19" extent="1-1"/>
+<wire x1="10.41" y1="44.6659" x2="19.09445" y2="30.13" width="0" layer="19" extent="1-1"/>
+<wire x1="0" y1="46.77" x2="10.41" y2="44.6659" width="0" layer="19" extent="1-1"/>
 </signal>
 <signal name="N$1">

Commit message: change lcd connector to vertical, remove lcd wire pads, correct connection for flash chips OE
Parts:
- removed 5V, 5V0, DB0, DB1, DB2, DB3, DB4, DB5, DB6, DB7, E, K, RS, RW, V0, VSS: TPTP07SQ, testpad:TP07SQ
- J1: value SM20B-SRDS-G-TF(LF)(SN) -> BM20B-SRDS-G-TF(LF)(SN); device SM20B-SRDS-G-TFLFSN:SM20BSRDSGTFLFSN -> BM20B-SRDS-G-TFLFSN:BM20BSRDSGTFLFSN
- moved J1 0.80 mm to (21.6, 3.81)
Connections:
- removed net VSS: J1.1, VSS.TP
- net +3V3: no longer J1.22
- net +5V: no longer 5V.TP, 5V0.TP
- net DB0: no longer DB0.TP
- net DB1: no longer DB1.TP
- net DB2: no longer DB2.TP
- net DB3: no longer DB3.TP
- net DB4: no longer DB4.TP
- net DB5: no longer DB5.TP
- net DB6: no longer DB6.TP
- net DB7: no longer DB7.TP
- net E: no longer E.TP
- net GND: now also J1.1
- net K: no longer K.TP
- net MNFLCE#: no longer U3.32
- net OE#: now also U3.32
- net RS: no longer RS.TP
- net RW: no longer RW.TP
- net VO: no longer V0.TP
