File: OpenX3/untitled.sch (EAGLE design)
At the start: 20 parts, among them J1 SM20B-SRDS-G-TF(LF)(SN), U1 LC4256V-75TN100CTQFP100-L, U2 AM29F016D-70EF

Commit message: more work
Parts:
- added J2: SM12B-SRSS-TB(LF)(SN), SM12B-SRSS-TB:SM12B-SRSS-TB(LF)(SN)
- added J3: 53398-0271, Molex 2 pos 53398-0271:53398-0271
- added J4: 1734260-3, TE 3 pos 1734260-3:1734260-3
- added LED1: (no value), adafruit:LEDCHIPLED_0805
- added R1, R2, R3, R4: UM6K31NFHATCNTRANS_UM6J1-L, UM6K31NFHA:UM6K31NFHATCNTRANS_UM6J1-L
- added R10: 200, SparkFun-Resistors:200OHM-0603-1/10W-1%
- added R5, R6, R8: 10k, SparkFun-Resistors:10KOHM-0603-1/10W-1%
- added R7: 0, SparkFun-Resistors:0OHM-0603-1/10W-5%
- added RN1, RN2: 10k, resistor-dil:4R-N0603-ARV
- added RN3: 100, resistor-dil:4R-N0603-ARV
- added U3: SST39SF020A-55-4C-WHE, SST39SF020A-55-4C-WHE:SST39SF020A-55-4C-WHE
Connections:
- net N$1 renamed A19
- net N$26 renamed OE#
- net N$3 renamed LAD2
- net N$34 renamed A20
- net N$39 renamed VSS
- net N$4 renamed LAD1
- net N$40 renamed VO
- net N$41 renamed RW
- net N$42 renamed DB0
- net N$46 renamed A
- net N$47 renamed VDD
- net N$48 renamed RS
- net N$49 renamed E
- net N$5 renamed LAD0
- net N$6 renamed LAD3
- net N$7 renamed A18
- removed net N$10: U1.A1, U2.A15
- removed net N$11: U1.A2, U2.A14
- removed net N$12: U1.A3, U2.A13
- removed net N$13: U1.A4, U2.A12
- removed net N$14: U1.B12, U2.CE#
- removed net N$15: U1.A5, U2.A11
- removed net N$16: U1.A6, U2.A10
- removed net N$18: U1.A8, U2.A8
- removed net N$19: U1.A9, U2.A7
- removed net N$20: U1.A10, U2.A6
- removed net N$21: U1.A11, U2.A5
- removed net N$22: U1.A12, U2.A4
- removed net N$23: U1.A13, U2.A3
- removed net N$24: U1.A14, U2.A2
- removed net N$25: U1.A15, U2.A1
- removed net N$27: U1.I_2, U2.DQ0
- removed net N$28: U1.D8, U2.DQ1
- removed net N$30: U1.C14, U2.DQ4
- removed net N$31: U1.C15, U2.DQ3
- removed net N$32: U1.C13, U2.DQ5
- removed net N$33: U1.C7, U2.DQ6
- removed net N$35: U1.VCCO_2, U2.A0
- removed net N$36: U1.B14, U2.WE#
- removed net N$38: U1.C6, U2.DQ7
- removed net N$43: J1.9, PAD9.P
- removed net N$44: J1.11, PAD11.P
- removed net N$45: J1.13, PAD13.P
- removed net N$50: J1.8, PAD8.P
- removed net N$51: J1.10, PAD10.P
- removed net N$52: J1.12, PAD12.P
- removed net N$53: J1.14, PAD14.P
- removed net N$54: J1.16, PAD16.P
- removed net N$8: U1.D0/GOE1, U2.A17
- removed net N$9: U1.A0/GOE0, U2.A16
- new net 3V3: JP1.9, R5.2, R6.1
- new net A0: U1.VCCO_2, U2.A0, U3.A0
- new net A1: U1.A15, U2.A1, U3.A1
- new net A10: U1.A6, U2.A10, U3.A10
- new net A11: U1.A5, U2.A11, U3.A11
- new net A12: U1.A4, U2.A12, U3.A12
- new net A13: U1.A3, U2.A13, U3.A13
- new net A14: U1.A2, U2.A14, U3.A14
- new net A15: U1.A1, U2.A15, U3.A15
- new net A16: U1.A0/GOE0, U2.A16, U3.A16
- new net A17: U1.D0/GOE1, U2.A17, U3.A17
- new net A2: U1.A14, U2.A2, U3.A2
- new net A3: U1.A13, U2.A3, U3.A3
- new net A4: U1.A12, U2.A4, U3.A4
- new net A5: U1.A11, U2.A5, U3.A5
- new net A6: U1.A10, U2.A6, U3.A6
- new net A7: U1.A9, U2.A7, U3.A7
- new net A8: U1.A8, U2.A8, U3.A8
- new net BLUELED: J2.8, RN3B.2
- new net BUFLCE#: U1.B11, U3.!CE
- new net D0: J4.1, JP1.4, R2.1
- new net DB1: J1.8, PAD8.P, U1.D11
- new net DB2: J1.9, PAD9.P, U1.D12
- new net DB3: J1.10, PAD10.P, U1.D13
- new net DB4: J1.11, PAD11.P, U1.C12
- new net DB5: J1.12, PAD12.P, U1.C8
- new net DB6: J1.13, PAD13.P, U1.C5
- new net DB7: J1.14, PAD14.P, U1.C4
- new net DQ0: U1.D7, U2.DQ0, U3.DQ0
- new net DQ1: U1.D8, U2.DQ1, U3.DQ1
- new net DQ3: U1.C15, U2.DQ3, U3.DQ3
- new net DQ4: U1.C14, U2.DQ4, U3.DQ4
- new net DQ5: U1.C13, U2.DQ5, U3.DQ5
- new net DQ6: U1.C7, U2.DQ6, U3.DQ6
- new net DQ7: U1.C6, U2.DQ7, U3.DQ7
- new net EXTPROTSW: J2.12, R8.1, U1.I_2
- new net FPEJECT: J3.1, R1.5
- new net FPPWR: J3.2, R1.2
- new net GND: J2.2, LED1.C
- new net HDDACT: J4.2, R3.5, RN1C.1, RN1C.2
- new net HDDLED: J2.9, RN3C.2
- new net K: J1.16, PAD16.P, R2.4
- new net LANACT: J4.3, R3.2, RN1D.1, RN1D.2
- new net LANLED: J2.10, RN3D.2
- new net MNFLCE#: U1.B12, U2.CE#, U3.!OE
- new net N$3: R10.1, R8.2
- new net N$4: R3.1, R3.4, R4.1, R4.4, R7.2, RN2A.1, RN2B.1, RN2C.1, RN2D.1
- new net N$5: LED1.A, R10.2
- new net N$56: R1.3, R1.6
- new net N$59: R1.4, R5.1, U1.CLK2/I
- new net N$61: R1.1, R6.2, U1.C0
- new net N$62: R2.2, U1.B8
- new net N$63: R2.5, U1.B10
- new net N$65: R2.3, R2.6, U1.GND_4
- new net N$70: R4.5, RN1B.2
- new net N$71: R4.2, RN1A.2
- new net N$72: R3.6, RN3D.1
- new net N$73: R3.3, RN3C.1
- new net N$74: R4.3, RN3B.1
- new net N$75: R4.6, RN3A.1
- new net N$78: RN1A.1, U1.B4
- new net N$79: RN1B.1, U1.B5
- new net N$87: J2.1, R7.1
- new net REDLED: J2.7, RN3A.2
- new net SWBANK1: J2.6, RN2D.2, U1.I_3
- new net SWBANK2: J2.5, RN2C.2, U1.I_4
- new net SWBANK3: J2.4, RN2B.2, U1.B7
- new net SWBANK4: J2.3, RN2A.2, U1.B6
- new net WE#: U1.B14, U2.WE#, U3.!WE
- net N$17: now also U3.A9
- net N$29: now also U3.DQ2
Other:
- moved on the sheet: J1, JP1, PAD1, PAD10, PAD11, PAD12, PAD13, PAD14, PAD15, PAD16, PAD2, PAD3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

Commit message: more work
Parts:
- added C1, C2: (no value), Wurth_Elektronik_Passive_Capacitors_rev18b:WCAP-CSGP_0603_885012006001_REFLOW
- added IC1: 24AA256SN, microchip:24AA256SN
- added LED2: (no value), adafruit:LEDCHIPLED_0805
- added R11: RV100F-30-4K1B-B10K-B301, RV100F-30-4K1B-B10K-B301:RV100F-30-4K1B-B10K-B301
- added R12: 4.7k, SparkFun-Resistors:4.7KOHM-0603-1/10W-1%
- added R9: 200, SparkFun-Resistors:200OHM-0603-1/10W-1%
- added S1: AYZ0102AGRLC, AYZ0102AGRLC:AYZ0102AGRLC
- renumbered PAD1 to VSS, PAD10 to DB3, PAD11 to DB4, PAD12 to DB5, PAD13 to DB6, PAD14 to DB7, PAD15 to 5V, PAD16 to K, PAD2 to 5V0, PAD3 to V0, PAD4 to RS, PAD5 to RW, PAD6 to E, PAD7 to DB0, PAD8 to DB1, PAD9 to DB2
Connections:
- removed net 3V3: JP1.9, R5.2, R6.1
- removed net A: 5V.P, J1.15
- removed net N$2: JP1.15, U1.VCCO_3
- removed net N$3: R10.1, R8.2
- removed net N$37: U2.RESET#, U2.VCC
- removed net VDD: 5V0.P, J1.2
- new net +3V3: C1.1, C2.1, IC1.VCC, JP1.15, JP1.9, R10.1, R5.2, R6.1, R8.2, U1.VCC, U1.VCCO, U1.VCCO_2, U1.VCCO_3, U1.VCCO_4, U1.VCCO_5, U1.VCCO_6, U1.VCC_2, U1.VCC_3, U1.VCC_4
- new net +5V: 5V.P, 5V0.P, J1.15, J1.2, JP1.6, R9.2, U2.RESET#, U2.VCC, U3.NC, U3.VDD
- new net LCLK: JP1.1, U1.CLK1/I
- new net N$1: LED2.A, R9.1
- new net SCL: IC1.SCL, JP1.13
- new net SDA: IC1.SDA, JP1.14
- net A0: now also U1.B15; no longer U1.VCCO_2
- net EXTPROTSW: now also S1.2
- net GND: now also C1.2, C2.2, IC1.GND, JP1.12, JP1.2, LED2.C, R11.3, R12.2, S1.3, U1.GND, U1.GND_10, U1.GND_11, U1.GND_12, U1.GND_2, U1.GND_3, U1.GND_5, U1.GND_6, U1.GND_7, U1.GND_8, U1.GND_9, U2.VSS, U3.VSS
- net OE#: now also U1.B14; no longer U1.B15
- net VO: now also R11.1, R11.2, R12.1
- net WE#: now also U1.B13; no longer U1.B14

Commit message: first attempt at pcb layout - having trouble routing
Parts:
- added JP2: (no value), pinhead:PINHD-1X1
- added JPA0, JPA1, JPA2, JPWP: JUMPER-SMT_3_NO_NO-SILK, SparkFun-Jumpers:JUMPER-SMT_3_NO_NO-SILK
- 5V, 5V0, DB0, DB1, DB2, DB3, DB4, DB5, DB6, DB7, E, K, RS, RW, V0, VSS: value WIREPADSMD1,27-254 -> TPTP07SQ; device wirepad:WIREPADSMD1,27-254 -> testpad:TPTP07SQ
- U3: value SST39SF020A-55-4C-WHE -> AM29F002BB90EI; device SST39SF020A-55-4C-WHE:SST39SF020A-55-4C-WHE -> AM29F002BB-90EI:AM29F002BB90EI
Connections:
- net N$17 renamed A9
- net N$29 renamed DQ2
- new net 3.3V: JPA0.3, JPA1.3, JPA2.3, JPWP.3
- new net EPA0: IC1.A0, JPA0.2
- new net EPA1: IC1.A1, JPA1.2
- new net EPA2: IC1.A2, JPA2.2
- new net EPWP: IC1.WP, JPWP.2
- new net TCK: J1.20, U1.TCK
- new net TDI: J1.18, U1.TDI
- new net TDO: J1.17, U1.TDO
- new net TMS: J1.19, U1.TMS
- net +3V3: now also C1.2, J1.22; no longer C1.1
- net +5V: now also 5V.TP, 5V0.TP, JP2.1, U3.!RESET, U3.VCC; no longer 5V.P, 5V0.P, U3.NC, U3.VDD
- net DB0: now also DB0.TP; no longer DB0.P
- net DB1: now also DB1.TP; no longer DB1.P
- net DB2: now also DB2.TP; no longer DB2.P
- net DB3: now also DB3.TP; no longer DB3.P
- net DB4: now also DB4.TP; no longer DB4.P
- net DB5: now also DB5.TP; no longer DB5.P
- net DB6: now also DB6.TP; no longer DB6.P
- net DB7: now also DB7.TP; no longer DB7.P
- net E: now also E.TP; no longer E.P
- net GND: now also C1.1, JPA0.1, JPA1.1, JPA2.1, JPWP.1; no longer C1.2
- net K: now also K.TP; no longer K.P
- net RS: now also RS.TP; no longer RS.P
- net RW: now also RW.TP; no longer RW.P
- net VO: now also V0.TP; no longer V0.P
- net VSS: now also VSS.TP; no longer VSS.P
Other:
- moved on the sheet: C1, IC1

Commit message: review ERC warnings; fix two missing junctions; one missing connection to GND on CPLD pin 18
Connections:
- removed net N$65: R2.3, R2.6, U1.GND_4
- net GND: now also R2.3, R2.6, U1.GND_4
Other:
- moved on the sheet: JPA0, JPA1, JPA2
Changed lines of the file:
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@@
 <attribute name="VALUE" x="167.64" y="-91.44" size="1.778" layer="96" rot="R270"/>
 </instance>
-<instance part="JPA0" gate="G$1" x="314.96" y="-119.38" smashed="yes" rot="R180">
-<attribute name="NAME" x="312.42" y="-119.761" size="1.778" layer="95" font="vector" rot="R180"/>
-<attribute name="VALUE" x="302.26" y="-118.999" size="1.778" layer="96" font="vector" rot="R180" align="top-left"/>
-</instance>
-<instance part="JPA1" gate="G$1" x="314.96" y="-106.68" smashed="yes" rot="R180">
-<attribute name="NAME" x="312.42" y="-107.061" size="1.778" layer="95" font="vector" rot="R180"/>
-</instance>
-<instance part="JPA2" gate="G$1" x="314.96" y="-93.98" smashed="yes" rot="R180">
-<attribute name="NAME" x="312.42" y="-94.361" size="1.778" layer="95" font="vector" rot="R180"/>
+<instance part="JPA0" gate="G$1" x="309.88" y="-119.38" smashed="yes" rot="R180">
+<attribute name="NAME" x="307.34" y="-119.761" size="1.778" layer="95" font="vector" rot="R180"/>
+</instance>
+<instance part="JPA1" gate="G$1" x="309.88" y="-106.68" smashed="yes" rot="R180">
+<attribute name="NAME" x="307.34" y="-107.061" size="1.778" layer="95" font="vector" rot="R180"/>
+</instance>
+<instance part="JPA2" gate="G$1" x="309.88" y="-93.98" smashed="yes" rot="R180">
+<attribute name="NAME" x="307.34" y="-94.361" size="1.778" layer="95" font="vector" rot="R180"/>
 </instance>
 <instance part="JPWP" gate="G$1" x="314.96" y="-81.28" smashed="yes" rot="R180">
@@
 <junction x="-149.86" y="106.68"/>
 <label x="-208.28" y="106.68" size="1.778" layer="95"/>
-</segment>
-</net>
-<net name="N$65" class="0">
-<segment>
-<pinref part="R2" gate="A" pin="3"/>
-<wire x1="-81.28" y1="104.14" x2="-81.28" y2="96.52" width="0.1524" layer="91"/>
-<wire x1="-81.28" y1="96.52" x2="-40.64" y2="96.52" width="0.1524" layer="91"/>
-<wire x1="-40.64" y1="96.52" x2="-40.64" y2="109.22" width="0.1524" layer="91"/>
-<pinref part="R2" gate="A" pin="6"/>
-<wire x1="-40.64" y1="109.22" x2="-45.72" y2="109.22" width="0.1524" layer="91"/>
-<pinref part="U1" gate="A" pin="GND_4"/>
-<wire x1="63.5" y1="20.32" x2="20.32" y2="20.32" width="0.1524" layer="91"/>
-<wire x1="20.32" y1="20.32" x2="20.32" y2="96.52" width="0.1524" layer="91"/>
-<wire x1="20.32" y1="96.52" x2="-40.64" y2="96.52" width="0.1524" layer="91"/>
-<junction x="-40.64" y="96.52"/>
 </segment>
 </net>
@@
 <wire x1="63.5" y1="48.26" x2="60.96" y2="48.26" width="0.1524" layer="91"/>
 <wire x1="60.96" y1="48.26" x2="58.42" y2="48.26" width="0.1524" layer="91"/>
-<wire x1="58.42" y1="48.26" x2="58.42" y2="0" width="0.1524" layer="91"/>
+<wire x1="58.42" y1="48.26" x2="58.42" y2="20.32" width="0.1524" layer="91"/>
 <junction x="58.42" y="0"/>
 <pinref part="U1" gate="A" pin="GND_2"/>
+<wire x1="58.42" y1="20.32" x2="58.42" y2="0" width="0.1524" layer="91"/>
 <wire x1="63.5" y1="63.5" x2="60.96" y2="63.5" width="0.1524" layer="91"/>
 <wire x1="60.96" y1="63.5" x2="60.96" y2="48.26" width="0.1524" layer="91"/>
@@
 <wire x1="27.94" y1="-43.18" x2="58.42" y2="-43.18" width="0.1524" layer="91"/>
 <junction x="58.42" y="-43.18"/>
+<pinref part="R2" gate="A" pin="3"/>
+<wire x1="-81.28" y1="104.14" x2="-81.28" y2="96.52" width="0.1524" layer="91"/>
+<wire x1="-81.28" y1="96.52" x2="-40.64" y2="96.52" width="0.1524" layer="91"/>
+<wire x1="-40.64" y1="96.52" x2="-40.64" y2="109.22" width="0.1524" layer="91"/>
+<pinref part="R2" gate="A" pin="6"/>
+<wire x1="-40.64" y1="109.22" x2="-45.72" y2="109.22" width="0.1524" layer="91"/>
+<pinref part="U1" gate="A" pin="GND_4"/>
+<wire x1="63.5" y1="20.32" x2="58.42" y2="20.32" width="0.1524" layer="91"/>
+<wire x1="58.42" y1="20.32" x2="20.32" y2="20.32" width="0.1524" layer="91"/>
+<wire x1="20.32" y1="20.32" x2="20.32" y2="96.52" width="0.1524" layer="91"/>
+<wire x1="20.32" y1="96.52" x2="-40.64" y2="96.52" width="0.1524" layer="91"/>
+<junction x="-40.64" y="96.52"/>
+<junction x="58.42" y="20.32"/>
 </segment>
 <segment>
@@
 <wire x1="317.5" y1="-111.76" x2="317.5" y2="-124.46" width="0.1524" layer="91"/>
 <wire x1="317.5" y1="-124.46" x2="317.5" y2="-137.16" width="0.1524" layer="91"/>
-<wire x1="314.96" y1="-99.06" x2="317.5" y2="-99.06" width="0.1524" layer="91"/>
+<wire x1="309.88" y1="-99.06" x2="317.5" y2="-99.06" width="0.1524" layer="91"/>
 <junction x="317.5" y="-99.06"/>
 <pinref part="JPA1" gate="G$1" pin="1"/>
-<wire x1="314.96" y1="-111.76" x2="317.5" y2="-111.76" width="0.1524" layer="91"/>
+<wire x1="309.88" y1="-111.76" x2="317.5" y2="-111.76" width="0.1524" layer="91"/>
 <junction x="317.5" y="-111.76"/>
 <pinref part="JPA0" gate="G$1" pin="1"/>
-<wire x1="314.96" y1="-124.46" x2="317.5" y2="-124.46" width="0.1524" layer="91"/>
+<wire x1="309.88" y1="-124.46" x2="317.5" y2="-124.46" width="0.1524" layer="91"/>
 <junction x="317.5" y="-124.46"/>
 <pinref part="SUPPLY10" gate="GND" pin="GND"/>
@@
 <segment>
 <pinref part="JPA2" gate="G$1" pin="2"/>
-<wire x1="320.04" y1="-93.98" x2="322.58" y2="-93.98" width="0.1524" layer="91"/>
+<wire x1="314.96" y1="-93.98" x2="322.58" y2="-93.98" width="0.1524" layer="91"/>
 <wire x1="322.58" y1="-93.98" x2="322.58" y2="-73.66" width="0.1524" layer="91"/>
 <pinref part="IC1" gate="G$1" pin="A2"/>
@@
 <segment>
 <pinref part="JPA1" gate="G$1" pin="2"/>
-<wire x1="320.04" y1="-106.68" x2="325.12" y2="-106.68" width="0.1524" layer="91"/>
+<wire x1="314.96" y1="-106.68" x2="325.12" y2="-106.68" width="0.1524" layer="91"/>
 <pinref part="IC1" gate="G$1" pin="A1"/>
 <wire x1="325.12" y1="-106.68" x2="325.12" y2="-76.2" width="0.1524" layer="91"/>
@@
 <segment>
 <pinref part="JPA0" gate="G$1" pin="2"/>
-<wire x1="320.04" y1="-119.38" x2="327.66" y2="-119.38" width="0.1524" layer="91"/>
+<wire x1="314.96" y1="-119.38" x2="327.66" y2="-119.38" width="0.1524" layer="91"/>
 <wire x1="327.66" y1="-119.38" x2="327.66" y2="-78.74" width="0.1524" layer="91"/>
 <pinref part="IC1" gate="G$1" pin="A0"/>
@@
 <wire x1="304.8" y1="-101.6" x2="304.8" y2="-114.3" width="0.1524" layer="91"/>
 <wire x1="304.8" y1="-137.16" x2="304.8" y2="-114.3" width="0.1524" layer="91"/>
-<wire x1="304.8" y1="-114.3" x2="314.96" y2="-114.3" width="0.1524" layer="91"/>
+<wire x1="304.8" y1="-114.3" x2="309.88" y2="-114.3" width="0.1524" layer="91"/>
 <pinref part="JPA1" gate="G$1" pin="3"/>
-<wire x1="314.96" y1="-101.6" x2="304.8" y2="-101.6" width="0.1524" layer="91"/>
+<wire x1="309.88" y1="-101.6" x2="304.8" y2="-101.6" width="0.1524" layer="91"/>
 <junction x="304.8" y="-101.6"/>
 <pinref part="JPA2" gate="G$1" pin="3"/>
-<wire x1="314.96" y1="-88.9" x2="304.8" y2="-88.9" width="0.1524" layer="91"/>
+<wire x1="309.88" y1="-88.9" x2="304.8" y2="-88.9" width="0.1524" layer="91"/>
 <junction x="304.8" y="-88.9"/>
 <pinref part="SUPPLY11" gate="G$1" pin="3.3V"/>
-</segment>
-</net>
+<junction x="304.8" y="-114.3"/>
+</segment>
+</net>

Commit message: change lcd connector to vertical, remove lcd wire pads, correct connection for flash chips OE
Parts:
- removed 5V, 5V0, DB0, DB1, DB2, DB3, DB4, DB5, DB6, DB7, E, K, RS, RW, V0, VSS: TPTP07SQ, testpad:TPTP07SQ
- J1: value SM20B-SRDS-G-TF(LF)(SN) -> BM20B-SRDS-G-TF(LF)(SN); device SM20B-SRDS-G-TFLFSN:SM20B-SRDS-G-TF(LF)(SN) -> BM20B-SRDS-G-TFLFSN:BM20B-SRDS-G-TF(LF)(SN)
Connections:
- removed net VSS: J1.1, VSS.TP
- net +3V3: no longer J1.22
- net +5V: no longer 5V.TP, 5V0.TP
- net DB0: no longer DB0.TP
- net DB1: no longer DB1.TP
- net DB2: no longer DB2.TP
- net DB3: no longer DB3.TP
- net DB4: no longer DB4.TP
- net DB5: no longer DB5.TP
- net DB6: no longer DB6.TP
- net DB7: no longer DB7.TP
- net E: no longer E.TP
- net GND: now also J1.1
- net K: no longer K.TP
- net MNFLCE#: no longer U3.!OE
- net OE#: now also U3.!OE
- net RS: no longer RS.TP
- net RW: no longer RW.TP
- net VO: no longer V0.TP
Other:
- moved on the sheet: JPWP
