File: OpenX3/openx3.brd (EAGLE design)
At the start: 46.7 x 49.1 mm, 34 parts, among them IC1 24AA256SN, J1 BM20B-SRDS-G-TF(LF)(SN), J2 SM12B-SRSS-TB(LF)(SN), J3 53398-0271, J4 1734260-3, U1 LC4256V-75TN100CTQFP100-L, U2 AM29F016D-70EF, U3 AM29F002BB90EI

Commit message: routing complete... passes DRC
Parts:
- moved JPWP 4.35 mm to (41.6, 28.2)
- moved JPA0 4.24 mm to (41.4, 22.4)
- moved JPA1 4.10 mm to (41.4, 24.4)
- moved JPA2 4.08 mm to (41.5, 26.5)
- moved J4 0.27 mm to (40.6, 42.7)
- moved IC1 0.13 mm to (40.7, 24.4)
- moved J3 0.13 mm to (34.0, 1.40)
Routing:
- net TDO: track 0.00 -> 44.2 mm, vias 0 -> 8
- net RW: track 0.00 -> 42.5 mm, vias 0 -> 4
- net DB4: track 1.49 -> 39.1 mm, vias 1 -> 4
- net RS: track 0.00 -> 35.6 mm, vias 0 -> 4
- net DB6: track 5.79 -> 36.8 mm, vias 1 -> 4
- net DB7: track 0.00 -> 29.3 mm, vias 0 -> 4
- net N$61: track 5.65 -> 33.4 mm, vias 0 -> 2
- net TMS: track 19.5 -> 46.4 mm, vias 1 -> 6
- net TDI: track 1.88 -> 24.4 mm, vias 1 -> 5
- net +3V3: track 136.6 -> 153.1 mm, vias 11 -> 10
- net DB5: track 16.9 -> 33.1 mm, vias 1 -> 4
- net SDA: track 0.00 -> 12.6 mm
- net SCL: track 0.00 -> 10.8 mm
- net N$4: track 21.2 -> 31.9 mm
- net DB2: track 44.8 -> 54.8 mm, vias 2 -> 4
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Other:
- board size 46.7 x 49.1 mm -> 46.9 x 49.8 mm

Commit message: Add files via upload
Parts:
- added U$1: (no value), OXC_Library:KEKULE-0002
Routing:
- net GND: track 6.86 -> 1.12 mm
Other:
- board size 46.9 x 49.8 mm -> 47 x 49.5 mm
Changed lines of the file:
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@@
 <?xml version="1.0" encoding="utf-8"?>
 <!DOCTYPE eagle SYSTEM "eagle.dtd">
-<eagle version="9.3.1">
+<eagle version="9.5.2">
 <drawing>
 <settings>
-<setting alwaysvectorfont="no"/>
+<setting alwaysvectorfont="yes"/>
 <setting verticaltext="up"/>
 </settings>
-<grid distance="1" unitdist="mil" unit="mil" style="lines" multiple="1" display="no" altdistance="5" altunitdist="mil" altunit="mil"/>
+<grid distance="0.127" unitdist="mm" unit="mm" style="lines" multiple="1" display="yes" altdistance="5" altunitdist="mil" altunit="mil"/>
 <layers>
 <layer number="1" name="Top" color="4" fill="1" visible="yes" active="yes"/>
-<layer number="2" name="Route2" color="16" fill="1" visible="no" active="yes"/>
-<layer number="3" name="Route3" color="17" fill="1" visible="no" active="yes"/>
-<layer number="4" name="Route4" color="18" fill="1" visible="no" active="yes"/>
-<layer number="5" name="Route5" color="19" fill="1" visible="no" active="yes"/>
-<layer number="6" name="Route6" color="25" fill="1" visible="no" active="yes"/>
-<layer number="7" name="Route7" color="26" fill="1" visible="no" active="yes"/>
-<layer number="8" name="Route8" color="27" fill="1" visible="no" active="yes"/>
-<layer number="9" name="Route9" color="28" fill="1" visible="no" active="yes"/>
-<layer number="10" name="Route10" color="29" fill="1" visible="no" active="yes"/>
-<layer number="11" name="Route11" color="30" fill="1" visible="no" active="yes"/>
-<layer number="12" name="Route12" color="20" fill="1" visible="no" active="yes"/>
-<layer number="13" name="Route13" color="21" fill="1" visible="no" active="yes"/>
-<layer number="14" name="Route14" color="22" fill="1" visible="no" active="yes"/>
-<layer number="15" name="Route15" color="23" fill="1" visible="yes" active="yes"/>
+<layer number="2" name="Route2" color="16" fill="1" visible="no" active="no"/>
+<layer number="3" name="Route3" color="17" fill="1" visible="no" active="no"/>
+<layer number="4" name="Route4" color="18" fill="1" visible="no" active="no"/>
+<layer number="5" name="Route5" color="19" fill="1" visible="no" active="no"/>
+<layer number="6" name="Route6" color="25" fill="1" visible="no" active="no"/>
+<layer number="7" name="Route7" color="26" fill="1" visible="no" active="no"/>
+<layer number="8" name="Route8" color="27" fill="1" visible="no" active="no"/>
+<layer number="9" name="Route9" color="28" fill="1" visible="no" active="no"/>
+<layer number="10" name="Route10" color="29" fill="1" visible="no" active="no"/>
+<layer number="11" name="Route11" color="30" fill="1" visible="no" active="no"/>
+<layer number="12" name="Route12" color="20" fill="1" visible="no" active="no"/>
+<layer number="13" name="Route13" color="21" fill="1" visible="no" active="no"/>
+<layer number="14" name="Route14" color="22" fill="1" visible="no" active="no"/>
+<layer number="15" name="Route15" color="23" fill="1" visible="no" active="no"/>
 <layer number="16" name="Bottom" color="1" fill="1" visible="yes" active="yes"/>
 <layer number="17" name="Pads" color="2" fill="1" visible="yes" active="yes"/>
@@
 <board>
 <plain>
-<wire x1="-1.27" y1="-1.27" x2="45.679409375" y2="-1.397" width="0" layer="20"/>
-<wire x1="45.679409375" y1="-1.397" x2="45.679409375" y2="48.233609375" width="0" layer="20"/>
-<wire x1="45.679409375" y1="48.233609375" x2="-1.27" y2="48.360609375" width="0" layer="20"/>
-<wire x1="-1.27" y1="48.360609375" x2="-1.27" y2="-1.27" width="0" layer="20"/>
+<wire x1="-1.27" y1="-1.27" x2="45.72" y2="-1.27" width="0" layer="20"/>
+<wire x1="45.72" y1="-1.27" x2="45.679409375" y2="48.233609375" width="0" layer="20"/>
+<wire x1="45.679409375" y1="48.233609375" x2="-1.27" y2="48.26" width="0" layer="20"/>
+<wire x1="-1.27" y1="48.26" x2="-1.27" y2="-1.27" width="0" layer="20"/>
 <text x="38.1" y="19.05" size="0.6096" layer="22" rot="MR270">GND</text>
 <text x="35.56" y="19.05" size="0.6096" layer="22" rot="MR270">VCC</text>
@@
 <attribute name="MOUSER_PRICE-STOCK" value="" x="21.59" y="3.81" size="1.778" layer="27" display="off"/>
 </element>
+<element name="U$1" library="OXC_Library" library_urn="urn:adsk.eagle:library:16553167" package="KEKULE-0002" package3d_urn="urn:adsk.eagle:package:16553233/1" value="" x="12.7" y="-0.508" smashed="yes" rot="MR0"/>
 </elements>
 <signals>
@@
 <via x="36.8046" y="14.7574" extent="1-16" drill="0.35"/>
 <via x="32.512" y="22.352" extent="1-16" drill="0.35"/>
-<wire x1="29.05125" y1="33.02" x2="28.9842" y2="33.12795" width="0.1524" layer="1"/>
-<wire x1="29.05125" y1="33.02" x2="28.98418125" y2="33.02" width="0.1524" layer="1"/>
 <via x="9.8806" y="36.576" extent="1-16" drill="0.35"/>
 <via x="9.9822" y="31.0134" extent="1-16" drill="0.35"/>
@@
 <via x="5.334" y="34.7218" extent="1-16" drill="0.35"/>
 <via x="3.9878" y="44.5008" extent="1-16" drill="0.35"/>
-<wire x1="28.4842" y1="17.97685" x2="28.4842" y2="19.137" width="0.1524" layer="1"/>
-<wire x1="28.4842" y1="19.137" x2="28.5242" y2="19.177" width="0.1524" layer="1"/>
 <via x="26.289" y="20.4216" extent="1-16" drill="0.35"/>
 <via x="23.876" y="24.6634" extent="1-16" drill="0.35"/>
@@
 <via x="30.861" y="24.384" extent="1-16" drill="0.35"/>
 <via x="31.115" y="32.0294" extent="1-16" drill="0.35"/>
-<wire x1="31.115" y1="32.0294" x2="31.115" y2="28.68815625" width="0.1524" layer="16"/>
-<wire x1="31.115" y1="28.68815625" x2="30.9908" y2="28.56395625" width="0.1524" layer="16"/>
-<wire x1="30.9908" y1="28.56395625" x2="30.9908" y2="28.244625" width="0.1524" layer="16"/>
-<wire x1="30.9908" y1="28.244625" x2="30.78201875" y2="28.03584375" width="0.1524" layer="16"/>
-<wire x1="30.78201875" y1="28.03584375" x2="30.78201875" y2="27.8623125" width="0.1524" layer="16"/>
-<wire x1="30.78201875" y1="27.8623125" x2="30.7848" y2="27.85953125" width="0.1524" layer="16"/>
-<wire x1="30.7848" y1="27.85953125" x2="30.7848" y2="27.8384" width="0.1524" layer="16"/>
 </signal>
 <signal name="N$1">
