File: OpenX3_rev2/openx3_rev2.sch (EAGLE design)
At the start: 33 parts, among them IC1 24AA256SN, J1 BM20B-SRDS-G-TF(LF)(SN), J2 SM12B-SRSS-TB(LF)(SN), J3 53398-0271, J4 1734260-3, U1 LC4256V-75TN100CTQFP100-L, U2 AM29F016D-70EF, U3 AM29F002BB90EI

Commit message: minor fixes to traces, but no changes, adding gerber file for 2nd pcb order with fixed 3v3 and gnd
Connections:
- net BLUELEDACT renamed N$6
- net BLUELED_O renamed N$74
- net D0_O renamed D0
- net LANACT_O renamed LANLED_O
- net REDLEDACT renamed N$71
- net REDLED_O renamed N$75
- removed net BLUELED_I: RN1B.1
- removed net DO_CTRL: R2.5
- removed net FPEJECT: R1.1, R6.2
- removed net FPPWR: R1.4, R5.1
- removed net HDDACT_0: R3.3
- removed net HDDACT_O: RN3C.1
- removed net K_PWM: R2.2
- removed net N$56: R1.3, R1.6
- removed net REDLED_I: RN1A.1
- removed net SWBABK3: RN2B.2
- new net HDDLED_O: R3.3, RN3C.1
- new net N$62: R2.2, U1.B8
- new net N$63: R2.5, U1.B10
- net A4: no longer U3.A4
- net A5: no longer U3.A5
- net A7: now also U3.A5
- net A8: now also U3.A4
- net GND: now also R1.3, R1.6
- net N$59: now also R1.4, R5.1
- net N$61: now also R1.1, R6.2
- net N$78: now also RN1A.1
- net N$79: now also RN1B.1
- net SWBANK3: now also RN2B.2
Other:
- moved on the sheet: J3, J4, LED2, R1, R2, R3, R4, R5, R6, R9, RN1A, RN1B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
